Commit message: Remove link collision macro

File: config/utils.xacro (robot description, xacro)
@@ -10,14 +10,4 @@
       <axis xyz="0 0 1" />
     </joint>
-  </xacro:macro>
-  <!-- Store collision type as a link for the collision object -->
-  <xacro:macro name="object_link_" params="name frame_id *geometry">
-    <link name="${name}">
-      <collision>
-        <geometry>
-          <xacro:insert_block name="geometry" />
-        </geometry>
-      </collision>
-    </link>
   </xacro:macro>
   <!-- Add dummy link with no collision -->

Commit message: Add subframes support for meshes
A node can be passed as an argument which will create all available
subframes for a mesh.

File: config/utils.xacro (robot description, xacro)
@@ -18,6 +18,24 @@
     </xacro:tf>
   </xacro:macro>
+  <!-- Add subframes for mesh -->
+  <xacro:macro name="loopmeshsubframes" params="current:=0 max:=^ node:=^ name:=^">
+    <xacro:if value="${max > current}">
+      <xacro:property name="xyz" value="0 0 0" />
+      <xacro:property name="rpy" value="0 0 0" />
+      <xacro:if value="${'xyz' in node[current]}">
+        <xacro:property name="xyz" value="${node[current]['xyz'][0]} ${node[current]['xyz'][1]} ${node[current]['xyz'][2]}" />
+      </xacro:if>>
+      <xacro:if value="${'rpy' in node[current]}">
+        <xacro:property name="rpy" value="${node[current]['rpy'][0]} ${node[current]['rpy'][1]} ${node[current]['rpy'][2]}" />
+      </xacro:if>>
+      <xacro:subframe name="${name}"
+                      subframe="${node[current]['name']}"
+                      frame_id="${name}"
+                      xyz="${xyz}" rpy="${rpy}" />
+      <xacro:loopmeshsubframes current="${current+1}"/>
+    </xacro:if>
+  </xacro:macro>
   <!-- Add mesh -->
-  <xacro:macro name="framemesh" params="name frame_id resource xyz:='0 0 0' rpy:='0 0 0' scale:='1.0 1.0 1.0'">
+  <xacro:macro name="framemesh" params="name frame_id resource xyz:='0 0 0' subframes:=false  rpy:='0 0 0' scale:='1.0 1.0 1.0'">
     <link name="${name}">
       <collision>
@@ -30,4 +48,7 @@
       <origin xyz="${xyz}" rpy="${rpy}"/>
     </xacro:tf>
+    <xacro:if value="${subframes}">
+      <xacro:loopmeshsubframes max="${len(subframes)}" node="${subframes}"/>
+    </xacro:if>
   </xacro:macro>
   <!-- Add primitive box -->

Commit message: Change mesh subframes node as a dict

File: config/utils.xacro (robot description, xacro)
@@ -19,16 +19,16 @@
   </xacro:macro>
   <!-- Add subframes for mesh -->
-  <xacro:macro name="loopmeshsubframes" params="current:=0 max:=^ node:=^ name:=^">
+  <xacro:macro name="loopmeshsubframes" params="current:=0 max:=^ node:=^ sorted_keys:=^ name:=^">
     <xacro:if value="${max > current}">
       <xacro:property name="xyz" value="0 0 0" />
       <xacro:property name="rpy" value="0 0 0" />
-      <xacro:if value="${'xyz' in node[current]}">
-        <xacro:property name="xyz" value="${node[current]['xyz'][0]} ${node[current]['xyz'][1]} ${node[current]['xyz'][2]}" />
+      <xacro:if value="${'xyz' in node[sorted_keys[current]]}">
+        <xacro:property name="xyz" value="${node[sorted_keys[current]]['xyz'][0]} ${node[sorted_keys[current]]['xyz'][1]} ${node[sorted_keys[current]]['xyz'][2]}" />
       </xacro:if>>
-      <xacro:if value="${'rpy' in node[current]}">
-        <xacro:property name="rpy" value="${node[current]['rpy'][0]} ${node[current]['rpy'][1]} ${node[current]['rpy'][2]}" />
+      <xacro:if value="${'rpy' in node[sorted_keys[current]]}">
+        <xacro:property name="rpy" value="${node[sorted_keys[current]]['rpy'][0]} ${node[sorted_keys[current]]['rpy'][1]} ${node[sorted_keys[current]]['rpy'][2]}" />
       </xacro:if>>
       <xacro:subframe name="${name}"
-                      subframe="${node[current]['name']}"
+                      subframe="${sorted_keys[current]}"
                       frame_id="${name}"
                       xyz="${xyz}" rpy="${rpy}" />
@@ -49,5 +49,5 @@
     </xacro:tf>
     <xacro:if value="${subframes}">
-      <xacro:loopmeshsubframes max="${len(subframes)}" node="${subframes}"/>
+      <xacro:loopmeshsubframes max="${len(subframes)}" node="${subframes}" sorted_keys="${sorted(subframes)}"/>
     </xacro:if>
   </xacro:macro>
