Commit message: Simplify shelf parameters

File: config/shelf.urdf.xacro (robot description, xacro)
@@ -9,16 +9,16 @@
                                     rpy:='0 0 0'
                                     board_number:=5
-                                    board_dim_x:=0.6
-                                    board_dim_y:=1.5
-                                    board_dim_z:=0.02
-                                    post_dim_x:=0.035
-                                    post_dim_y:=0.035
-                                    post_dim_z:=1.25
+                                    board_dimensions:='0.6 1.5 0.02'
+                                    post_dimensions:='0.035 0.035 1.25'
                                     dl:=_">
   <!-- Property -->
   <xacro:property name="root" value="${name}" />
-  <xacro:property name="board_dimensions" value="${board_dim_x} ${board_dim_y} ${board_dim_z}" />
-  <xacro:property name="post_dimensions" value="${post_dim_x} ${post_dim_y} ${post_dim_z}" />
   <xacro:property name="board_gap" value="${post_dim_z/(board_number)}" />
+  <xacro:property name="board_dim_x" value="${board_dimensions.split()[0]}" />
+  <xacro:property name="board_dim_y" value="${board_dimensions.split()[1]}" />
+  <xacro:property name="board_dim_z" value="${board_dimensions.split()[2]}" />
+  <xacro:property name="post_dim_x" value="${post_dimensions.split()[0]}" />
+  <xacro:property name="post_dim_y" value="${post_dimensions.split()[1]}" />
+  <xacro:property name="post_dim_z" value="${post_dimensions.split()[2]}" />
   <!-- Subframes -->
   <xacro:macro name="loop_subframe" params="current:=0
@@ -39,19 +39,19 @@
   <!-- Shelf posts -->
   <xacro:framebox name="${root}${dl}post_bl"
-             frame_id="${root}"
-             dimensions="${post_dimensions}"
-             xyz="${-(board_dim_x/2 - post_dim_x/2)} ${-(board_dim_y/2 - post_dim_y/2)}   ${post_dim_z/2}" />
+                  frame_id="${root}"
+                  dimensions="${post_dimensions}"
+                  xyz="${-(board_dim_x/2 - post_dim_x/2)} ${-(board_dim_y/2 - post_dim_y/2)}   ${post_dim_z/2}" />
   <xacro:framebox name="${root}${dl}post_br"
-             frame_id="${root}${dl}post_bl"
-             dimensions="${post_dimensions}"
-             xyz="0 ${board_dim_y - post_dim_y} 0"/>
+                  frame_id="${root}${dl}post_bl"
+                  dimensions="${post_dimensions}"
+                  xyz="0 ${board_dim_y - post_dim_y} 0"/>
   <xacro:framebox name="${root}${dl}post_fl"
-             frame_id="${root}${dl}post_bl"
-             dimensions="${post_dimensions}"
-             xyz="${board_dim_x - post_dim_x} 0 0"/>
+                  frame_id="${root}${dl}post_bl"
+                  dimensions="${post_dimensions}"
+                  xyz="${board_dim_x - post_dim_x} 0 0"/>
   <xacro:framebox name="${root}${dl}post_fr"
-             frame_id="${root}${dl}post_fl"
-             dimensions="${post_dimensions}"
-             xyz="0 ${board_dim_y - post_dim_y} 0"/>
+                  frame_id="${root}${dl}post_fl"
+                  dimensions="${post_dimensions}"
+                  xyz="0 ${board_dim_y - post_dim_y} 0"/>
   <!-- Shelf boards -->
   <xacro:macro name="loop_board" params="current:=0

Commit message: Refactor urdf link parser
Enables loading a robot URDF into collision objects. Fixes potential
segfault when arbitrary URDF file where loaded.

File: config/shelf.urdf.xacro (robot description, xacro)
@@ -28,5 +28,5 @@
                       subframe="level${current+1}"
                       frame_id="${root}${dl}board${current+1}"
-                      xyz="0 0 0" />
+                      xyz="0 0 ${board_dim_z/2}" />
       <xacro:loop_subframe current="${current+1}"/>
     </xacro:if>
@@ -59,7 +59,7 @@
     <xacro:if value="${max > current}">
       <xacro:framebox name="${root}${dl}board${current+1}"
-                 frame_id="${root}"
-                 dimensions="${board_dimensions}"
-                 xyz="0 0 ${(current+1)*board_gap - board_dim_z/2}"/>
+                      frame_id="${root}"
+                      dimensions="${board_dimensions}"
+                      xyz="0 0 ${(current+1)*board_gap - board_dim_z/2}"/>
       <xacro:loop_board current="${current+1}"/>
     </xacro:if>

File: config/utils.xacro (robot description, xacro)
@@ -35,6 +35,4 @@
     <link name="${name}">
       <collision>
-        <!-- define frame at bottom of geometry -->
-        <origin xyz="${xyz.split()[0]} ${xyz.split()[1]} ${float(xyz.split()[2]) + float(dimensions.split()[2])}" />
         <geometry>
           <box size="${dimensions}" />

Commit message: Refactor shelf tag to add vertical boards

File: config/shelf.urdf.xacro (robot description, xacro)
@@ -8,49 +8,74 @@
                                     xyz:='0 0 0'
                                     rpy:='0 0 0'
-                                    board_number:=5
-                                    board_dimensions:='0.6 1.5 0.02'
-                                    post_dimensions:='0.035 0.035 1.25'
+                                    dimensions:='0.6 1.5 1.25'
+                                    h_boards:=5
+                                    v_boards:=3
+                                    h_board_thickness:=0.02
+                                    v_board_thickness:=0.02
+                                    back_board:=false
                                     dl:=_">
   <!-- Property -->
   <xacro:property name="root" value="${name}" />
-  <xacro:property name="board_gap" value="${post_dim_z/(board_number)}" />
-  <xacro:property name="board_dim_x" value="${board_dimensions.split()[0]}" />
-  <xacro:property name="board_dim_y" value="${board_dimensions.split()[1]}" />
-  <xacro:property name="board_dim_z" value="${board_dimensions.split()[2]}" />
-  <xacro:property name="post_dim_x" value="${post_dimensions.split()[0]}" />
-  <xacro:property name="post_dim_y" value="${post_dimensions.split()[1]}" />
-  <xacro:property name="post_dim_z" value="${post_dimensions.split()[2]}" />
+  <xacro:property name="hboard_gap" value="${float(dimensions.split()[2])/h_boards}" />
+  <xacro:property name="vboard_gap" value="${float(dimensions.split()[1])/(1 + v_boards)}" />
+  <xacro:property name="dim_x" value="${dimensions.split()[0]}" />
+  <xacro:property name="dim_y" value="${dimensions.split()[1]}" />
+  <xacro:property name="dim_z" value="${dimensions.split()[2]}" />
+  <xacro:property name="hboard_dim_x" value="${dim_x}" />
+  <xacro:property name="hboard_dim_y" value="${vboard_gap + v_board_thickness/2}" />
+  <xacro:property name="hboard_dim_z" value="${h_board_thickness}" />
+  <xacro:property name="hboard_dimensions" value="${hboard_dim_x} ${hboard_dim_y} ${hboard_dim_z}" />
+  <xacro:property name="vboard_dim_x" value="${dim_x}" />
+  <xacro:property name="vboard_dim_y" value="${v_board_thickness}" />
+  <xacro:property name="vboard_dim_z" value="${dim_z}" />
+  <xacro:property name="vboard_dimensions" value="${vboard_dim_x} ${vboard_dim_y} ${vboard_dim_z}" />
   <!-- Base link -->
   <xacro:dummy name="${root}"
                frame_id="${frame_id}"
                xyz="${xyz}" rpy="${rpy}" />
-  <!-- Shelf posts -->
-  <xacro:framebox name="${root}${dl}post_bl"
+  <!-- Leftmost and rightmost vertical boards -->
+  <xacro:framebox name="${root}${dl}vboard1"
                   frame_id="${root}"
-                  dimensions="${post_dimensions}"
-                  xyz="${-(board_dim_x/2 - post_dim_x/2)} ${-(board_dim_y/2 - post_dim_y/2)}  0" />
-  <xacro:framebox name="${root}${dl}post_br"
-                  frame_id="${root}${dl}post_bl/bottom"
-                  dimensions="${post_dimensions}"
-                  xyz="0 ${board_dim_y - post_dim_y} 0"/>
-  <xacro:framebox name="${root}${dl}post_fl"
-                  frame_id="${root}${dl}post_bl/bottom"
-                  dimensions="${post_dimensions}"
-                  xyz="${board_dim_x - post_dim_x} 0 0"/>
-  <xacro:framebox name="${root}${dl}post_fr"
-                  frame_id="${root}${dl}post_fl/bottom"
-                  dimensions="${post_dimensions}"
-                  xyz="0 ${board_dim_y - post_dim_y} 0"/>
-  <!-- Shelf boards -->
-  <xacro:macro name="loop_board" params="current:=0 max:=^">
+                  dimensions="${vboard_dimensions}"
+                  xyz="0 ${-(dim_y/2 - v_board_thickness/2)} 0"/>
+  <xacro:framebox name="${root}${dl}vboard${v_boards + 2}"
+                  frame_id="${root}"
+                  dimensions="${vboard_dimensions}"
+                  xyz="0 ${dim_y/2 - v_board_thickness/2} 0"/>
+  <!-- Vertical inside boards -->
+  <xacro:macro name="loopvboard" params="current:=0 max:=^">
     <xacro:if value="${max > current}">
-      <xacro:framebox name="${root}${dl}board${current+1}"
-                 frame_id="${root}"
-                 dimensions="${board_dimensions}"
-                 xyz="0 0 ${(current+1)*board_gap - board_dim_z}"/>
-      <xacro:loop_board current="${current+1}"/>
+      <xacro:framebox name="${root}${dl}vboard${current+2}"
+                      frame_id="${root}${dl}vboard1/bottom"
+                      dimensions="${vboard_dimensions}"
+                      xyz="0 ${(current+1)*vboard_gap- v_board_thickness/2} 0"/>
+      <xacro:loopvboard current="${current+1}"/>
     </xacro:if>
   </xacro:macro>
-  <xacro:loop_board max="${board_number}"/>
+  <xacro:loopvboard max="${v_boards}"/>
+  <!-- Horizontal boards -->
+  <xacro:macro name="loophboard" params="current:=0 index:=^ max:=^">
+    <xacro:if value="${max > current}">
+      <xacro:framebox name="${root}${dl}board${index*h_boards+current+1}"
+                 frame_id="${root}${dl}vboard${index+1}/bottom"
+                 dimensions="${hboard_dimensions}"
+                 xyz="0 ${(vboard_gap - v_board_thickness/2)/2} ${(current + 1)*hboard_gap - h_board_thickness}"/>
+      <xacro:loophboard current="${current+1}"/>
+    </xacro:if>
+  </xacro:macro>
+  <xacro:macro name="loophrowboard" params="current:=0 max:=^">
+    <xacro:if value="${max > current}">
+      <xacro:loophboard index="${current}" max="${h_boards}"/>
+      <xacro:loophrowboard current="${current+1}"/>
+    </xacro:if>
+  </xacro:macro>
+  <xacro:loophrowboard max="${v_boards + 1}"/>
+  <!-- Back board -->
+  <xacro:if value="${back_board}">
+    <xacro:framebox name="${root}${dl}backboard"
+                    frame_id="${root}"
+                    dimensions="${v_board_thickness} ${dim_y} ${dim_z}"
+                    xyz="${-dim_x/2} 0 0"/>
+  </xacro:if>
   </xacro:macro>
 </robot>

Commit message: avoid variable named "max"
This triggers the following warning in xacro lately:

> redefining global symbol: max

it's obviously not a good idea to override the python max function :)

File: config/shelf.urdf.xacro (robot description, xacro)
@@ -44,6 +44,6 @@
                   xyz="0 ${dim_y/2 - v_board_thickness/2} 0"/>
   <!-- Vertical inside boards -->
-  <xacro:macro name="loopvboard" params="current:=0 max:=^">
-    <xacro:if value="${max > current}">
+  <xacro:macro name="loopvboard" params="current:=0 until:=^">
+    <xacro:if value="${until > current}">
       <xacro:framebox name="${root}${dl}vboard${current+2}"
                       frame_id="${root}${dl}vboard1/bottom"
@@ -53,8 +53,8 @@
     </xacro:if>
   </xacro:macro>
-  <xacro:loopvboard max="${v_boards}"/>
+  <xacro:loopvboard until="${v_boards}"/>
   <!-- Horizontal boards -->
-  <xacro:macro name="loophboard" params="current:=0 index:=^ max:=^">
-    <xacro:if value="${max > current}">
+  <xacro:macro name="loophboard" params="current:=0 index:=^ until:=^">
+    <xacro:if value="${until > current}">
       <xacro:framebox name="${root}${dl}board${index*h_boards+current+1}"
                  frame_id="${root}${dl}vboard${index+1}/bottom"
@@ -64,11 +64,11 @@
     </xacro:if>
   </xacro:macro>
-  <xacro:macro name="loophrowboard" params="current:=0 max:=^">
-    <xacro:if value="${max > current}">
-      <xacro:loophboard index="${current}" max="${h_boards}"/>
+  <xacro:macro name="loophrowboard" params="current:=0 until:=^">
+    <xacro:if value="${until > current}">
+      <xacro:loophboard index="${current}" until="${h_boards}"/>
       <xacro:loophrowboard current="${current+1}"/>
     </xacro:if>
   </xacro:macro>
-  <xacro:loophrowboard max="${v_boards + 1}"/>
+  <xacro:loophrowboard until="${v_boards + 1}"/>
   <!-- Back board -->
   <xacro:if value="${back_board}">

File: config/utils.xacro (robot description, xacro)
@@ -19,6 +19,6 @@
   </xacro:macro>
   <!-- Add subframes for mesh -->
-  <xacro:macro name="loopmeshsubframes" params="current:=0 max:=^ node:=^ sorted_keys:=^ name:=^">
-    <xacro:if value="${max > current}">
+  <xacro:macro name="loopmeshsubframes" params="current:=0 until:=^ node:=^ sorted_keys:=^ name:=^">
+    <xacro:if value="${until > current}">
       <xacro:property name="xyz" value="0 0 0" />
       <xacro:property name="rpy" value="0 0 0" />
@@ -49,5 +49,5 @@
     </xacro:tf>
     <xacro:if value="${'subframes' in metadata}">
-      <xacro:loopmeshsubframes max="${len(metadata['subframes'])}" node="${metadata['subframes']}" sorted_keys="${sorted(metadata['subframes'])}"/>
+      <xacro:loopmeshsubframes until="${len(metadata['subframes'])}" node="${metadata['subframes']}" sorted_keys="${sorted(metadata['subframes'])}"/>
     </xacro:if>
   </xacro:macro>
