Commit message: Change package name

File: config/opencrate.urdf.xacro (robot description, xacro)
@@ -1,5 +1,5 @@
 <?xml version="1.0" ?>
 <robot name="opencrate" xmlns:xacro="http://www.ros.org/wiki/xacro">
-  <xacro:include filename="$(find scene_parser)/config/utils.xacro" />
+  <xacro:include filename="$(find urdf_to_scene)/config/utils.xacro" />
   <!-- Generic open crate macro -->
   <xacro:macro name="opencrate" params="name

File: config/scene.urdf.xacro (robot description, xacro)
@@ -1,8 +1,8 @@
 <?xml version="1.0" ?>
 <robot name="scene" xmlns:xacro="http://www.ros.org/wiki/xacro">
-  <xacro:include filename="$(find scene_parser)/config/utils.xacro" />
-  <xacro:include filename="$(find scene_parser)/config/shelf.urdf.xacro" />
+  <xacro:include filename="$(find urdf_to_scene)/config/utils.xacro" />
+  <xacro:include filename="$(find urdf_to_scene)/config/shelf.urdf.xacro" />
   <!-- Import object metadata -->
-  <xacro:include filename="$(find scene_parser)/mesh/metadata.xacro" />
+  <xacro:include filename="$(find urdf_to_scene)/mesh/metadata.xacro" />
   <link name="world" />
   <!-- Create default shelf -->

File: config/shelf.urdf.xacro (robot description, xacro)
@@ -1,5 +1,5 @@
 <?xml version="1.0" ?>
 <robot name="shelf" xmlns:xacro="http://www.ros.org/wiki/xacro">
-  <xacro:include filename="$(find scene_parser)/config/utils.xacro" />
+  <xacro:include filename="$(find urdf_to_scene)/config/utils.xacro" />
   <!-- Generic Open Shelf macro -->
   <!-- TODO add option for an open and a closed shelf -->

File: mesh/metadata.xacro (robot description, xacro)
@@ -2,5 +2,5 @@
 <robot xmlns:xacro="http://www.ros.org/wiki/xacro" name="metadata">
   <!-- Load metadata of all meshes -->
-  <xacro:property name="pkg_path"   value="$(find scene_parser)/mesh/"/>
+  <xacro:property name="pkg_path"   value="$(find urdf_to_scene)/mesh/"/>
   <xacro:property name="can"   value="${load_yaml(pkg_path + 'can.yaml')['can']}"/>
 </robot>
