Commit message: Refactor package

File: config/scene.urdf.xacro (robot description, xacro)
@@ -5,15 +5,15 @@
   <link name="world" />
   <!-- Create default shelf -->
-  <xacro:shelf name="book-shelf"
+  <xacro:shelf name="book_shelf"
                frame_id="world"
                xyz="0.8 0 0"/>
   <!-- Add cube on book-shelf level-1 -->
   <xacro:box name="box"
-             frame_id="book-shelf/level-1"
+             frame_id="book_shelf/level1"
              xyz="0 0 0.005"
              dimensions="0.03 0.03 0.03"/>
   <!-- Add can on book-shelf level-2 -->
   <xacro:mesh name="can"
-              frame_id="book-shelf/level-2"
+              frame_id="book_shelf/level2"
               scale="0.01 0.01 0.01"
               resource="package://scene_parser/mesh/can.stl"/>

File: config/shelf.urdf.xacro (robot description, xacro)
@@ -2,65 +2,68 @@
 <robot name="shelf" xmlns:xacro="http://www.ros.org/wiki/xacro">
   <xacro:include filename="$(find scene_parser)/config/utils.xacro" />
+  <!-- Generic Open Shelf macro -->
+  <!-- TODO add option for an open and a closed shelf -->
   <xacro:macro name="shelf" params="name
                                     frame_id
                                     xyz:='0 0 0'
                                     rpy:='0 0 0'
-                                    shelf_number:=5
-                                    shelf_dim_x:=0.6
-                                    shelf_dim_y:=1.5
-                                    shelf_dim_z:=0.02
+                                    board_number:=5
+                                    board_dim_x:=0.6
+                                    board_dim_y:=1.5
+                                    board_dim_z:=0.02
                                     post_dim_x:=0.035
                                     post_dim_y:=0.035
-                                    post_dim_z:=1.25">
+                                    post_dim_z:=1.25
+                                    dl:=_">
   <!-- Property -->
-  <xacro:property name="base_link" value="${name}" />
-  <xacro:property name="dl" value="_" />
-  <xacro:property name="shelf_dimensions" value="${shelf_dim_x} ${shelf_dim_y} ${shelf_dim_z}" />
+  <xacro:property name="root" value="${name}" />
+  <xacro:property name="board_dimensions" value="${board_dim_x} ${board_dim_y} ${board_dim_z}" />
   <xacro:property name="post_dimensions" value="${post_dim_x} ${post_dim_y} ${post_dim_z}" />
-  <xacro:property name="shelf_gap" value="${post_dim_z/(shelf_number)}" />
-  <!-- Subframes wrt. base_link -->
+  <xacro:property name="board_gap" value="${post_dim_z/(board_number)}" />
+  <!-- Subframes -->
   <xacro:macro name="loop_subframe" params="current:=0
                                          max:=^">
     <xacro:if value="${max > current}">
-      <xacro:subframe name="${name}"
-                      subframe="level-${current+1}"
-                      xyz="0 0 ${(current+1)*shelf_gap}" />
+      <xacro:subframe name="${root}"
+                      subframe="level${current+1}"
+                      frame_id="${root}${dl}board${current+1}"
+                      xyz="0 0 0" />
       <xacro:loop_subframe current="${current+1}"/>
     </xacro:if>
   </xacro:macro>
-  <xacro:loop_subframe max="${shelf_number}"/>
+  <xacro:loop_subframe max="${board_number}"/>
   <!-- Base link -->
-  <xacro:dummy name="${base_link}"
+  <xacro:dummy name="${root}"
                frame_id="${frame_id}"
                xyz="${xyz}" rpy="${rpy}" />
   <!-- Shelf posts -->
-  <xacro:box name="${name}${dl}post_bl"
-             frame_id="${base_link}"
+  <xacro:box name="${root}${dl}post_bl"
+             frame_id="${root}"
              dimensions="${post_dimensions}"
-             xyz="${-(shelf_dim_x/2 - post_dim_x/2)} ${-(shelf_dim_y/2 - post_dim_y/2)}   ${post_dim_z/2}" />
-  <xacro:box name="${name}${dl}post_br"
-             frame_id="${name}${dl}post_bl"
+             xyz="${-(board_dim_x/2 - post_dim_x/2)} ${-(board_dim_y/2 - post_dim_y/2)}   ${post_dim_z/2}" />
+  <xacro:box name="${root}${dl}post_br"
+             frame_id="${root}${dl}post_bl"
              dimensions="${post_dimensions}"
-             xyz="0 ${shelf_dim_y - post_dim_y} 0"/>
-  <xacro:box name="${name}${dl}post_fl"
-             frame_id="${name}${dl}post_bl"
+             xyz="0 ${board_dim_y - post_dim_y} 0"/>
+  <xacro:box name="${root}${dl}post_fl"
+             frame_id="${root}${dl}post_bl"
              dimensions="${post_dimensions}"
-             xyz="${shelf_dim_x - post_dim_x} 0 0"/>
-  <xacro:box name="${name}${dl}post_fr"
-             frame_id="${name}${dl}post_fl"
+             xyz="${board_dim_x - post_dim_x} 0 0"/>
+  <xacro:box name="${root}${dl}post_fr"
+             frame_id="${root}${dl}post_fl"
              dimensions="${post_dimensions}"
-             xyz="0 ${shelf_dim_y - post_dim_y} 0"/>
-  <!-- Shelf -->
-  <xacro:macro name="loop_shelf" params="current:=0
+             xyz="0 ${board_dim_y - post_dim_y} 0"/>
+  <!-- Shelf boards -->
+  <xacro:macro name="loop_board" params="current:=0
                                          max:=^">
     <xacro:if value="${max > current}">
-      <xacro:box name="${name}${dl}${current+1}"
-                 frame_id="${base_link}"
-                 dimensions="${shelf_dimensions}"
-                 xyz="0 0 ${(current+1)*shelf_gap - shelf_dim_z/2}"/>
-      <xacro:loop_shelf current="${current+1}"/>
+      <xacro:box name="${root}${dl}board${current+1}"
+                 frame_id="${root}"
+                 dimensions="${board_dimensions}"
+                 xyz="0 0 ${(current+1)*board_gap - board_dim_z/2}"/>
+      <xacro:loop_board current="${current+1}"/>
     </xacro:if>
   </xacro:macro>
-  <xacro:loop_shelf max="${shelf_number}"/>
+  <xacro:loop_board max="${board_number}"/>
   </xacro:macro>
 </robot>

File: config/utils.xacro (robot description, xacro)
@@ -1,6 +1,7 @@
 <?xml version="1.0" ?>
 <robot xmlns:xacro="http://www.ros.org/wiki/xacro" name="panda">
-  <!-- Utility macros for collision objects -->
-  <xacro:macro name="add_joint" params="name frame_id *origin">
+  <!-- Utility macros for creating collision objects as URDF -->
+  <!-- Store tf information as a joint for the collision object -->
+  <xacro:macro name="object_joint_" params="name frame_id *origin">
     <joint name="${name}" type="fixed">
       <xacro:insert_block name="origin" />
@@ -10,5 +11,6 @@
     </joint>
   </xacro:macro>
-  <xacro:macro name="add_link" params="name frame_id *geometry">
+  <!-- Store collision type as a link for the collision object -->
+  <xacro:macro name="object_link_" params="name frame_id *geometry">
     <link name="${name}">
       <collision>
@@ -19,31 +21,43 @@
     </link>
   </xacro:macro>
+  <!-- Add dummy link with no collision -->
   <xacro:macro name="dummy" params="name frame_id xyz:='0 0 0' rpy:='0 0 0'">
     <link name="${name}"/>
-    <xacro:add_joint name="${name}" frame_id="${frame_id}">
+    <xacro:object_joint_ name="${name}" frame_id="${frame_id}">
       <origin xyz="${xyz}" rpy="${rpy}"/>
-    </xacro:add_joint>>
+    </xacro:object_joint_>>
   </xacro:macro>
+  <!-- Add mesh -->
   <xacro:macro name="mesh" params="name frame_id resource xyz:='0 0 0' rpy:='0 0 0' scale:='1.0 1.0 1.0'">
-    <xacro:add_link name="${name}" frame_id="${frame_id}">
+    <xacro:object_link_ name="${name}" frame_id="${frame_id}">
         <mesh filename="${resource}" scale="${scale}" />
-    </xacro:add_link>
-    <xacro:add_joint name="${name}" frame_id="${frame_id}">
+    </xacro:object_link_>
+    <xacro:object_joint_ name="${name}" frame_id="${frame_id}">
       <origin xyz="${xyz}" rpy="${rpy}"/>
-    </xacro:add_joint>
+    </xacro:object_joint_>
   </xacro:macro>
+  <!-- Add primitive box -->
   <xacro:macro name="box" params="name frame_id dimensions xyz:='0 0 0' rpy:='0 0 0'">
-    <xacro:add_link name="${name}" frame_id="${frame_id}">
+    <xacro:object_link_ name="${name}" frame_id="${frame_id}">
           <box size="${dimensions}" />
-    </xacro:add_link>
-    <xacro:add_joint name="${name}" frame_id="${frame_id}">
+    </xacro:object_link_>
+    <xacro:object_joint_ name="${name}" frame_id="${frame_id}">
       <origin xyz="${xyz}" rpy="${rpy}"/>
-    </xacro:add_joint>
+    </xacro:object_joint_>
   </xacro:macro>
-  <xacro:macro name="subframe" params="name subframe dl:=/ xyz:='0 0 0' rpy:='0 0 0'">
+  <!-- Add subframe -->
+  <!-- Optional: frame_id defaults to name parameter if empty -->
+  <xacro:macro name="subframe" params="name subframe frame_id:='' dl:=/ xyz:='0 0 0' rpy:='0 0 0'">
     <link name="${name}${dl}${subframe}"/>
-    <xacro:add_joint name="${name}${dl}${subframe}" frame_id="${name}">
-      <origin xyz="${xyz}" rpy="${rpy}"/>
-    </xacro:add_joint>
+    <xacro:if value="${len(frame_id) > 0}">
+      <xacro:object_joint_ name="${name}${dl}${subframe}" frame_id="${frame_id}">
+        <origin xyz="${xyz}" rpy="${rpy}"/>
+      </xacro:object_joint_>
+    </xacro:if>
+    <xacro:unless value="${len(frame_id) > 0}">
+      <xacro:object_joint_ name="${name}${dl}${subframe}" frame_id="${name}">
+        <origin xyz="${xyz}" rpy="${rpy}"/>
+      </xacro:object_joint_>
+    </xacro:unless>
   </xacro:macro>
 </robot>

Commit message: rename utility macros
box is already a urdf tag. In theory that's no problem, but xacro in melodic
still supports (with a warning) calling xacro macros without the `xacro:` prefix.

Why go for something cryptic like "object_joint_", when "tf" is perfectly correct :-)

File: config/scene.urdf.xacro (robot description, xacro)
@@ -9,10 +9,10 @@
                xyz="0.8 0 0"/>
   <!-- Add cube on book-shelf level-1 -->
-  <xacro:box name="box"
+  <xacro:framebox name="box"
              frame_id="book_shelf/level1"
              xyz="0 0 0.005"
              dimensions="0.03 0.03 0.03"/>
   <!-- Add can on book-shelf level-2 -->
-  <xacro:mesh name="can"
+  <xacro:framemesh name="can"
               frame_id="book_shelf/level2"
               scale="0.01 0.01 0.01"

File: config/shelf.urdf.xacro (robot description, xacro)
@@ -38,17 +38,17 @@
                xyz="${xyz}" rpy="${rpy}" />
   <!-- Shelf posts -->
-  <xacro:box name="${root}${dl}post_bl"
+  <xacro:framebox name="${root}${dl}post_bl"
              frame_id="${root}"
              dimensions="${post_dimensions}"
              xyz="${-(board_dim_x/2 - post_dim_x/2)} ${-(board_dim_y/2 - post_dim_y/2)}   ${post_dim_z/2}" />
-  <xacro:box name="${root}${dl}post_br"
+  <xacro:framebox name="${root}${dl}post_br"
              frame_id="${root}${dl}post_bl"
              dimensions="${post_dimensions}"
              xyz="0 ${board_dim_y - post_dim_y} 0"/>
-  <xacro:box name="${root}${dl}post_fl"
+  <xacro:framebox name="${root}${dl}post_fl"
              frame_id="${root}${dl}post_bl"
              dimensions="${post_dimensions}"
              xyz="${board_dim_x - post_dim_x} 0 0"/>
-  <xacro:box name="${root}${dl}post_fr"
+  <xacro:framebox name="${root}${dl}post_fr"
              frame_id="${root}${dl}post_fl"
              dimensions="${post_dimensions}"
@@ -58,5 +58,5 @@
                                          max:=^">
     <xacro:if value="${max > current}">
-      <xacro:box name="${root}${dl}board${current+1}"
+      <xacro:framebox name="${root}${dl}board${current+1}"
                  frame_id="${root}"
                  dimensions="${board_dimensions}"

File: config/utils.xacro (robot description, xacro)
@@ -3,8 +3,8 @@
   <!-- Utility macros for creating collision objects as URDF -->
   <!-- Store tf information as a joint for the collision object -->
-  <xacro:macro name="object_joint_" params="name frame_id *origin">
+  <xacro:macro name="tf" params="name parent *origin">
     <joint name="${name}" type="fixed">
       <xacro:insert_block name="origin" />
-      <parent link="${frame_id}" />
+      <parent link="${parent}" />
       <child link="${name}" />
       <axis xyz="0 0 1" />
@@ -24,25 +24,35 @@
   <xacro:macro name="dummy" params="name frame_id xyz:='0 0 0' rpy:='0 0 0'">
     <link name="${name}"/>
-    <xacro:object_joint_ name="${name}" frame_id="${frame_id}">
+    <xacro:tf name="${name}" parent="${frame_id}">
       <origin xyz="${xyz}" rpy="${rpy}"/>
-    </xacro:object_joint_>>
+    </xacro:tf>
   </xacro:macro>
   <!-- Add mesh -->
-  <xacro:macro name="mesh" params="name frame_id resource xyz:='0 0 0' rpy:='0 0 0' scale:='1.0 1.0 1.0'">
-    <xacro:object_link_ name="${name}" frame_id="${frame_id}">
-        <mesh filename="${resource}" scale="${scale}" />
-    </xacro:object_link_>
-    <xacro:object_joint_ name="${name}" frame_id="${frame_id}">
+  <xacro:macro name="framemesh" params="name frame_id resource xyz:='0 0 0' rpy:='0 0 0' scale:='1.0 1.0 1.0'">
+    <link name="${name}">
+      <collision>
+        <geometry>
+          <mesh filename="${resource}" scale="${scale}" />
+        </geometry>
+      </collision>
+    </link>
+    <xacro:tf name="${name}" parent="${frame_id}">
       <origin xyz="${xyz}" rpy="${rpy}"/>
-    </xacro:object_joint_>
+    </xacro:tf>
   </xacro:macro>
   <!-- Add primitive box -->
-  <xacro:macro name="box" params="name frame_id dimensions xyz:='0 0 0' rpy:='0 0 0'">
-    <xacro:object_link_ name="${name}" frame_id="${frame_id}">
+  <xacro:macro name="framebox" params="name frame_id dimensions xyz:='0 0 0' rpy:='0 0 0'">
+    <link name="${name}">
+      <collision>
+        <!-- define frame at bottom of geometry -->
+        <origin xyz="${xyz.split()[0]} ${xyz.split()[1]} ${float(xyz.split()[2]) + float(dimensions.split()[2])}" />
+        <geometry>
           <box size="${dimensions}" />
-    </xacro:object_link_>
-    <xacro:object_joint_ name="${name}" frame_id="${frame_id}">
+        </geometry>
+      </collision>
+    </link>
+    <xacro:tf name="${name}" parent="${frame_id}">
       <origin xyz="${xyz}" rpy="${rpy}"/>
-    </xacro:object_joint_>
+    </xacro:tf>
   </xacro:macro>
   <!-- Add subframe -->
@@ -51,12 +61,12 @@
     <link name="${name}${dl}${subframe}"/>
     <xacro:if value="${len(frame_id) > 0}">
-      <xacro:object_joint_ name="${name}${dl}${subframe}" frame_id="${frame_id}">
+      <xacro:tf name="${name}${dl}${subframe}" parent="${frame_id}">
         <origin xyz="${xyz}" rpy="${rpy}"/>
-      </xacro:object_joint_>
+      </xacro:tf>
     </xacro:if>
     <xacro:unless value="${len(frame_id) > 0}">
-      <xacro:object_joint_ name="${name}${dl}${subframe}" frame_id="${name}">
+      <xacro:tf name="${name}${dl}${subframe}" parent="${name}">
         <origin xyz="${xyz}" rpy="${rpy}"/>
-      </xacro:object_joint_>
+      </xacro:tf>
     </xacro:unless>
   </xacro:macro>

Commit message: Automate height of primitive wrt to bottom/top

File: config/scene.urdf.xacro (robot description, xacro)
@@ -7,13 +7,22 @@
   <xacro:shelf name="book_shelf"
                frame_id="world"
-               xyz="0.8 0 0"/>
+               xyz="0.8 0 0"
+               board_dimensions="0.6 1.5 0.02"/>
   <!-- Add cube on book-shelf level-1 -->
   <xacro:framebox name="box"
-             frame_id="book_shelf/level1"
-             xyz="0 0 0.005"
-             dimensions="0.03 0.03 0.03"/>
+             frame_id="book_shelf_board1/top"
+             xyz="0 0 0"
+             dimensions="0.05 0.05 0.12"/>
+  <xacro:framebox name="box1"
+             frame_id="book_shelf_post_bl/bottom"
+             xyz="0 0 0"
+             dimensions="0.05 0.05 0.12"/>
+  <xacro:framebox name="box2"
+             frame_id="book_shelf_post_bl/top"
+             xyz="0 0 0"
+             dimensions="0.05 0.05 0.12"/>
   <!-- Add can on book-shelf level-2 -->
   <xacro:framemesh name="can"
-              frame_id="book_shelf/level2"
+              frame_id="book_shelf_board5/top"
               scale="0.01 0.01 0.01"
               resource="package://scene_parser/mesh/can.stl"/>

File: config/shelf.urdf.xacro (robot description, xacro)
@@ -21,16 +21,4 @@
   <xacro:property name="post_dim_y" value="${post_dimensions.split()[1]}" />
   <xacro:property name="post_dim_z" value="${post_dimensions.split()[2]}" />
-  <!-- Subframes -->
-  <xacro:macro name="loop_subframe" params="current:=0
-                                         max:=^">
-    <xacro:if value="${max > current}">
-      <xacro:subframe name="${root}"
-                      subframe="level${current+1}"
-                      frame_id="${root}${dl}board${current+1}"
-                      xyz="0 0 0" />
-      <xacro:loop_subframe current="${current+1}"/>
-    </xacro:if>
-  </xacro:macro>
-  <xacro:loop_subframe max="${board_number}"/>
   <!-- Base link -->
   <xacro:dummy name="${root}"
@@ -41,15 +29,15 @@
                   frame_id="${root}"
                   dimensions="${post_dimensions}"
-                  xyz="${-(board_dim_x/2 - post_dim_x/2)} ${-(board_dim_y/2 - post_dim_y/2)}   ${post_dim_z/2}" />
+                  xyz="${-(board_dim_x/2 - post_dim_x/2)} ${-(board_dim_y/2 - post_dim_y/2)}  0" />
   <xacro:framebox name="${root}${dl}post_br"
-                  frame_id="${root}${dl}post_bl"
+                  frame_id="${root}${dl}post_bl/bottom"
                   dimensions="${post_dimensions}"
                   xyz="0 ${board_dim_y - post_dim_y} 0"/>
   <xacro:framebox name="${root}${dl}post_fl"
-                  frame_id="${root}${dl}post_bl"
+                  frame_id="${root}${dl}post_bl/bottom"
                   dimensions="${post_dimensions}"
                   xyz="${board_dim_x - post_dim_x} 0 0"/>
   <xacro:framebox name="${root}${dl}post_fr"
-                  frame_id="${root}${dl}post_fl"
+                  frame_id="${root}${dl}post_fl/bottom"
                   dimensions="${post_dimensions}"
                   xyz="0 ${board_dim_y - post_dim_y} 0"/>
@@ -61,5 +49,5 @@
                  frame_id="${root}"
                  dimensions="${board_dimensions}"
-                 xyz="0 0 ${(current+1)*board_gap - board_dim_z/2}"/>
+                 xyz="0 0 ${(current+1)*board_gap - board_dim_z}"/>
       <xacro:loop_board current="${current+1}"/>
     </xacro:if>

File: config/utils.xacro (robot description, xacro)
@@ -33,8 +33,13 @@
   <!-- Add primitive box -->
   <xacro:macro name="framebox" params="name frame_id dimensions xyz:='0 0 0' rpy:='0 0 0'">
+    <!-- Parent joint -->
+    <xacro:tf name="${name}" parent="${frame_id}">
+        <origin xyz="${xyz.split()[0]} ${xyz.split()[1]} ${float(xyz.split()[2]) + float(dimensions.split()[2])}" />
+    </xacro:tf>
+    <!-- Child link -->
     <link name="${name}">
       <collision>
         <!-- define frame at bottom of geometry -->
-        <origin xyz="${xyz.split()[0]} ${xyz.split()[1]} ${float(xyz.split()[2]) + float(dimensions.split()[2])}" />
+      <origin xyz="0 0 ${-float(dimensions.split()[2])/2}" rpy="${rpy}"/>
         <geometry>
           <box size="${dimensions}" />
@@ -42,7 +47,12 @@
       </collision>
     </link>
-    <xacro:tf name="${name}" parent="${frame_id}">
-      <origin xyz="${xyz}" rpy="${rpy}"/>
-    </xacro:tf>
+    <xacro:subframe name="${name}"
+                    subframe="bottom"
+                    frame_id="${name}"
+                    xyz="0 0 ${-float(dimensions.split()[2])/2}" />
+    <xacro:subframe name="${name}"
+                    subframe="top"
+                    frame_id="${name}"
+                    xyz="0 0 ${float(dimensions.split()[2])/2}" />
   </xacro:macro>
   <!-- Add subframe -->
