Commit message: Framebox tag tf defaults to center top of box
The tf of a framebox is now located at the top of the box. The visual of
the framebox is compensated because a primitive origin is wrt. the center.

File: config/scene.urdf.xacro (robot description, xacro)
@@ -5,15 +5,15 @@
   <link name="world" />
   <!-- Create default shelf -->
-  <xacro:shelf name="book_shelf"
+  <xacro:shelf name="bookshelf"
                frame_id="world"
                xyz="0.8 0 0"/>
   <!-- Add cube on book-shelf level-1 -->
   <xacro:framebox name="box"
-             frame_id="book_shelf/level1"
-             xyz="0 0 0.005"
+             frame_id="bookshelf_board1"
+             xyz="0 0 0"
              dimensions="0.03 0.03 0.03"/>
   <!-- Add can on book-shelf level-2 -->
   <xacro:framemesh name="can"
-              frame_id="book_shelf/level2"
+              frame_id="bookshelf_board5"
               scale="0.01 0.01 0.01"
               resource="package://scene_parser/mesh/can.stl"/>

File: config/shelf.urdf.xacro (robot description, xacro)
@@ -21,16 +21,4 @@
   <xacro:property name="post_dim_y" value="${post_dimensions.split()[1]}" />
   <xacro:property name="post_dim_z" value="${post_dimensions.split()[2]}" />
-  <!-- Subframes -->
-  <xacro:macro name="loop_subframe" params="current:=0
-                                         max:=^">
-    <xacro:if value="${max > current}">
-      <xacro:subframe name="${root}"
-                      subframe="level${current+1}"
-                      frame_id="${root}${dl}board${current+1}"
-                      xyz="0 0 ${board_dim_z/2}" />
-      <xacro:loop_subframe current="${current+1}"/>
-    </xacro:if>
-  </xacro:macro>
-  <xacro:loop_subframe max="${board_number}"/>
   <!-- Base link -->
   <xacro:dummy name="${root}"
@@ -41,25 +29,24 @@
                   frame_id="${root}"
                   dimensions="${post_dimensions}"
-                  xyz="${-(board_dim_x/2 - post_dim_x/2)} ${-(board_dim_y/2 - post_dim_y/2)}   ${post_dim_z/2}" />
+                  xyz="${-(board_dim_x/2 - post_dim_x/2)} ${-(board_dim_y/2 - post_dim_y/2)}  0" />
   <xacro:framebox name="${root}${dl}post_br"
-                  frame_id="${root}${dl}post_bl"
+                  frame_id="${root}${dl}post_bl/bottom"
                   dimensions="${post_dimensions}"
                   xyz="0 ${board_dim_y - post_dim_y} 0"/>
   <xacro:framebox name="${root}${dl}post_fl"
-                  frame_id="${root}${dl}post_bl"
+                  frame_id="${root}${dl}post_bl/bottom"
                   dimensions="${post_dimensions}"
                   xyz="${board_dim_x - post_dim_x} 0 0"/>
   <xacro:framebox name="${root}${dl}post_fr"
-                  frame_id="${root}${dl}post_fl"
+                  frame_id="${root}${dl}post_fl/bottom"
                   dimensions="${post_dimensions}"
                   xyz="0 ${board_dim_y - post_dim_y} 0"/>
   <!-- Shelf boards -->
-  <xacro:macro name="loop_board" params="current:=0
-                                         max:=^">
+  <xacro:macro name="loop_board" params="current:=0 max:=^">
     <xacro:if value="${max > current}">
       <xacro:framebox name="${root}${dl}board${current+1}"
-                      frame_id="${root}"
-                      dimensions="${board_dimensions}"
-                      xyz="0 0 ${(current+1)*board_gap - board_dim_z/2}"/>
+                 frame_id="${root}"
+                 dimensions="${board_dimensions}"
+                 xyz="0 0 ${(current+1)*board_gap - board_dim_z}"/>
       <xacro:loop_board current="${current+1}"/>
     </xacro:if>

File: config/utils.xacro (robot description, xacro)
@@ -33,6 +33,14 @@
   <!-- Add primitive box -->
   <xacro:macro name="framebox" params="name frame_id dimensions xyz:='0 0 0' rpy:='0 0 0'">
+    <!-- Parent joint -->
+    <xacro:tf name="${name}" parent="${frame_id}">
+      <!-- Add fixed origin and include z dimension -->
+      <origin xyz="${xyz.split()[0]} ${xyz.split()[1]} ${float(xyz.split()[2]) + float(dimensions.split()[2])}"/>
+    </xacro:tf>
+    <!-- Child link -->
     <link name="${name}">
       <collision>
+        <!-- Replace collision visualization because box origin is in the middle -->
+        <origin xyz="0 0 ${-float(dimensions.split()[2])/2}" rpy="${rpy}"/>
         <geometry>
           <box size="${dimensions}" />
@@ -40,7 +48,28 @@
       </collision>
     </link>
-    <xacro:tf name="${name}" parent="${frame_id}">
-      <origin xyz="${xyz}" rpy="${rpy}"/>
-    </xacro:tf>
+    <xacro:subframe name="${name}"
+                    subframe="bottom"
+                    frame_id="${name}"
+                    xyz="0 0 ${-float(dimensions.split()[2])}" />
+    <xacro:subframe name="${name}"
+                    subframe="top"
+                    frame_id="${name}"
+                    xyz="0 0 ${float(dimensions.split()[2])}" />
+    <xacro:subframe name="${name}"
+                    subframe="back"
+                    frame_id="${name}"
+                    xyz="${-float(dimensions.split()[0])/2} 0 0" />
+    <xacro:subframe name="${name}"
+                    subframe="front"
+                    frame_id="${name}"
+                    xyz="${float(dimensions.split()[0])/2} 0 0" />
+    <xacro:subframe name="${name}"
+                    subframe="left"
+                    frame_id="${name}"
+                    xyz="0 ${-float(dimensions.split()[1])/2} 0" />
+    <xacro:subframe name="${name}"
+                    subframe="right"
+                    frame_id="${name}"
+                    xyz="0 ${float(dimensions.split()[1])/2} 0" />
   </xacro:macro>
   <!-- Add subframe -->

Commit message: Refactor framemesh tag to support metadata

File: config/scene.urdf.xacro (robot description, xacro)
@@ -3,18 +3,20 @@
   <xacro:include filename="$(find scene_parser)/config/utils.xacro" />
   <xacro:include filename="$(find scene_parser)/config/shelf.urdf.xacro" />
+  <!-- Import object metadata -->
+  <xacro:include filename="$(find scene_parser)/mesh/metadata.xacro" />
   <link name="world" />
   <!-- Create default shelf -->
+  <!-- Subframes are automatically created -->
   <xacro:shelf name="bookshelf"
                frame_id="world"
                xyz="0.8 0 0"/>
-  <!-- Add cube on book-shelf level-1 -->
+  <!-- Add cube on bookshelf board1 -->
   <xacro:framebox name="box"
-             frame_id="bookshelf_board1"
-             xyz="0 0 0"
-             dimensions="0.03 0.03 0.03"/>
-  <!-- Add can on book-shelf level-2 -->
+                  frame_id="bookshelf_board1"
+                  xyz="0 0 0"
+                  dimensions="0.03 0.03 0.03"/>
+  <!-- Add can on bookshelf board5 -->
   <xacro:framemesh name="can"
-              frame_id="bookshelf_board5"
-              scale="0.01 0.01 0.01"
-              resource="package://scene_parser/mesh/can.stl"/>
+                   frame_id="bookshelf_board5"
+                   metadata="${can}"/>
 </robot>

File: config/utils.xacro (robot description, xacro)
@@ -28,5 +28,5 @@
       <xacro:if value="${'rpy' in node[sorted_keys[current]]}">
         <xacro:property name="rpy" value="${node[sorted_keys[current]]['rpy'][0]} ${node[sorted_keys[current]]['rpy'][1]} ${node[sorted_keys[current]]['rpy'][2]}" />
-      </xacro:if>>
+      </xacro:if>
       <xacro:subframe name="${name}"
                       subframe="${sorted_keys[current]}"
@@ -37,9 +37,9 @@
   </xacro:macro>
   <!-- Add mesh -->
-  <xacro:macro name="framemesh" params="name frame_id resource xyz:='0 0 0' subframes:=false  rpy:='0 0 0' scale:='1.0 1.0 1.0'">
+  <xacro:macro name="framemesh" params="name frame_id metadata xyz:='0 0 0' rpy:='0 0 0' scale:='1.0 1.0 1.0'">
     <link name="${name}">
       <collision>
         <geometry>
-          <mesh filename="${resource}" scale="${scale}" />
+          <mesh filename="${metadata['resource']}" scale="${scale}" />
         </geometry>
       </collision>
@@ -48,6 +48,6 @@
       <origin xyz="${xyz}" rpy="${rpy}"/>
     </xacro:tf>
-    <xacro:if value="${subframes}">
-      <xacro:loopmeshsubframes max="${len(subframes)}" node="${subframes}" sorted_keys="${sorted(subframes)}"/>
+    <xacro:if value="${'subframes' in metadata}">
+      <xacro:loopmeshsubframes max="${len(metadata['subframes'])}" node="${metadata['subframes']}" sorted_keys="${sorted(metadata['subframes'])}"/>
     </xacro:if>
   </xacro:macro>

Commit message: Speed test

File: config/scene.urdf.xacro (robot description, xacro)
@@ -20,3 +20,16 @@
                    frame_id="bookshelf_board5"
                    metadata="${can}"/>
+ <xacro:macro name="loop" params="items:=^">
+		<xacro:if value="${items}">
+			<!-- pop first item from list -->
+			<xacro:property name="item" value="${items.pop(0)}"/>
+      <!-- create multiple book shelves primitives -->
+      <xacro:shelf name="bookshelf${item}"
+                   frame_id="world"
+                   xyz="0.8 0 ${item}"/>
+			<!-- recursively call myself -->
+			<xacro:loop/>
+		</xacro:if>
+	</xacro:macro>
+	<xacro:loop items="${[1,2,3,4,5,6,7,8,9,10]}"/>
 </robot>

Commit message: cleanup

File: config/scene.urdf.xacro (robot description, xacro)
@@ -3,33 +3,17 @@
   <xacro:include filename="$(find urdf_to_scene)/config/utils.xacro" />
   <xacro:include filename="$(find urdf_to_scene)/config/shelf.urdf.xacro" />
-  <!-- Import object metadata -->
-  <xacro:include filename="$(find urdf_to_scene)/mesh/metadata.xacro" />
   <link name="world" />
-  <!-- Create default shelf -->
-  <!-- Subframes are automatically created -->
-  <xacro:shelf name="bookshelf"
-               frame_id="world"
-               xyz="0.8 0 0"/>
-  <!-- Add cube on bookshelf board1 -->
-  <xacro:framebox name="box"
-                  frame_id="bookshelf_board1"
-                  xyz="0 0 0"
-                  dimensions="0.03 0.03 0.03"/>
-  <!-- Add can on bookshelf board5 -->
-  <xacro:framemesh name="can"
-                   frame_id="bookshelf_board5"
-                   metadata="${can}"/>
- <xacro:macro name="loop" params="items:=^">
-		<xacro:if value="${items}">
-			<!-- pop first item from list -->
-			<xacro:property name="item" value="${items.pop(0)}"/>
-      <!-- create multiple book shelves primitives -->
+  <xacro:macro name="loop" params="items:=^">
+    <xacro:if value="${items}">
+      <!-- pop first item from list -->
+      <xacro:property name="item" value="${items.pop(0)}"/>
+      <!-- create multiple bookshelves (which is a collection of primitives) -->
       <xacro:shelf name="bookshelf${item}"
                    frame_id="world"
                    xyz="0.8 0 ${item}"/>
-			<!-- recursively call myself -->
-			<xacro:loop/>
-		</xacro:if>
-	</xacro:macro>
-	<xacro:loop items="${[1,2,3,4,5,6,7,8,9,10]}"/>
+      <!-- recursively call myself -->
+      <xacro:loop/>
+    </xacro:if>
+  </xacro:macro>
+  <xacro:loop items="${[1,2,3,4,5,6,7,8,9,10]}"/>
 </robot>
