Commit message: Reformat Xacro macro planning scene API
Add descriptive macro names and comments. Update object collection.

File: examples/scene.urdf.xacro (robot description, xacro)
@@ -3,20 +3,31 @@
   <xacro:include filename="$(find urdf_to_scene)/xacro/planning_scene.xacro" />
   <xacro:include filename="$(find urdf_to_scene)/xacro/collision_objects/shelf.urdf.xacro" />
-  <!-- Import object metadata -->
   <xacro:include filename="$(find urdf_to_scene)/mesh/metadata.xacro" />
-  <link name="world" />
+  <!-- Planning frame
+       1- Add a virtual frame, a static transform broadcaster must be supplied:
+           <link name="world"/>
+       2- Add the robot base link directly, e.g. for the panda:
+           <link name="panda_link0"/>
+       3- Use the xacro macro 'planning_fft' which will fill the PlanningScene 'fixed_frame_transforms':
+           <planning_fft name="panda_link0" parent="world" xyz="0 0 0"/>
+  -->
+  <link name="world"/>
+  <!-- Add the static transfrom manually -->
+  <planning_fft name="panda_link0"
+                parent="world"
+                xyz="0 0 0"/>
   <!-- Create default shelf -->
-  <!-- Subframes are automatically created -->
   <xacro:shelf name="bookshelf"
                frame_id="world"
-               xyz="0.8 0 0"/>
+               xyz="0.8 0 0"
+               h_board_thickness="0.02"/>
   <!-- Add cube on bookshelf board1 -->
-  <xacro:framebox name="box"
-                  frame_id="bookshelf_board1"
-                  xyz="0 0 0"
-                  dimensions="0.03 0.03 0.03"/>
+  <xacro:collision_box name="box"
+                       frame_id="bookshelf_board1/top"
+                       xyz="0 0 ${0.05/2}"
+                       dimensions="0.05 0.05 0.05"/>
   <!-- Add can on bookshelf board5 -->
-  <xacro:framemesh name="can"
-                   frame_id="bookshelf_board5"
-                   metadata="${can}"/>
+  <xacro:collision_mesh name="can"
+                        frame_id="bookshelf_board5/top"
+                        resource="${can.resource}"/>
 </robot>

File: xacro/collision_objects/opencrate.urdf.xacro (robot description, xacro)
@@ -1,49 +1,47 @@
 <?xml version="1.0" ?>
 <robot name="opencrate" xmlns:xacro="http://www.ros.org/wiki/xacro">
-  <xacro:include filename="$(find urdf_to_scene)/config/utils.xacro" />
-  <!-- Generic open crate macro -->
-  <xacro:macro name="opencrate" params="name
-                                        frame_id
-                                        xyz:='0 0 0'
-                                        rpy:='0 0 0'
-                                        dimensions:='1 1 1'
-                                        thickness:=0.1
-                                        dl:=_">
-  <!-- Property -->
-  <xacro:property name="root"  value="${name}" />
-  <xacro:property name="dim_x" value="${dimensions.split()[0]}" />
-  <xacro:property name="dim_y" value="${dimensions.split()[1]}" />
-  <xacro:property name="dim_z" value="${dimensions.split()[2]}" />
-  <!-- Base link -->
-  <xacro:dummy name="${root}"
-               frame_id="${frame_id}"
-               xyz="${xyz}" rpy="${rpy}" />
-  <!-- Individual boards -->
-  <xacro:framebox name="${root}${dl}bottom"
-                  frame_id="${root}"
-                  dimensions="${dim_x} ${dim_y} ${thickness}"
-                  xyz="0 0 0" />
-  <!--
-  <xacro:framebox name="${root}${dl}top"
-                  frame_id="${root}${dl}bottom"
-                  dimensions="${dim_x} ${dim_y} ${thickness}"
-                  xyz="0 0 ${dim_z - thickness}"/>
-  -->
-  <xacro:framebox name="${root}${dl}back"
-                  frame_id="${root}"
-                  dimensions="${thickness} ${dim_y} ${dim_z}"
-                  xyz="${-dim_x/2 + thickness/2} 0 0"/>
-  <xacro:framebox name="${root}${dl}front"
-                  frame_id="${root}${dl}back/bottom"
-                  dimensions="${thickness} ${dim_y} ${dim_z}"
-                  xyz="${dim_x - thickness} 0 0"/>
-  <xacro:framebox name="${root}${dl}left"
-                  frame_id="${root}"
-                  dimensions="${dim_x} ${thickness} ${dim_z}"
-                  xyz="0 ${-dim_y/2 + thickness/2} 0"/>
-  <xacro:framebox name="${root}${dl}right"
-                  frame_id="${root}${dl}left/bottom"
-                  dimensions="${dim_x} ${thickness} ${dim_z}"
-                  xyz="0 ${dim_y - thickness} 0"/>
-  </xacro:macro>
+    <xacro:include filename="$(find urdf_to_scene)/xacro/planning_scene.xacro" />
+    <!-- Generic open crate macro -->
+    <xacro:macro name="opencrate" params="name
+                                          frame_id
+                                          xyz:='0 0 0'
+                                          rpy:='0 0 0'
+                                          dimensions:='0.3 0.3 0.2'
+                                          thickness:=0.01
+                                          dl:=_">
+    <!-- Property -->
+    <xacro:property name="root"  value="${name}" />
+    <xacro:property name="dim_x" value="${dimensions.split()[0]}" />
+    <xacro:property name="dim_y" value="${dimensions.split()[1]}" />
+    <xacro:property name="dim_z" value="${dimensions.split()[2]}" />
+    <!-- Base link -->
+    <xacro:frame name="${root}"
+                frame_id="${frame_id}"
+                xyz="${xyz}" rpy="${rpy}" />
+    <!-- Individual boards -->
+    <xacro:collision_box name="${root}${dl}bottom"
+                         frame_id="${root}"
+                         dimensions="${dim_x} ${dim_y} ${thickness}"
+                         xyz="0 0 ${thickness/2}" />
+    <!-- <xacro:collision_box name="${root}${dl}top" -->
+    <!--                 frame_id="${root}${dl}bottom" -->
+    <!--                 dimensions="${dim_x} ${dim_y} ${thickness}" -->
+    <!--                 xyz="0 0 ${dim_z - thickness}"/> -->
+    <xacro:collision_box name="${root}${dl}back"
+                         frame_id="${root}"
+                         dimensions="${thickness} ${dim_y} ${dim_z}"
+                         xyz="${-dim_x/2 + thickness/2} 0 ${dim_z/2}"/>
+    <xacro:collision_box name="${root}${dl}front"
+                         frame_id="${root}${dl}back/bottom"
+                         dimensions="${thickness} ${dim_y} ${dim_z}"
+                         xyz="${dim_x - thickness} 0 ${dim_z/2}"/>
+    <xacro:collision_box name="${root}${dl}left"
+                         frame_id="${root}"
+                         dimensions="${dim_x} ${thickness} ${dim_z}"
+                         xyz="0 ${-dim_y/2 + thickness/2} ${dim_z/2}"/>
+    <xacro:collision_box name="${root}${dl}right"
+                         frame_id="${root}${dl}left/bottom"
+                         dimensions="${dim_x} ${thickness} ${dim_z}"
+                         xyz="0 ${dim_y - thickness} ${dim_z/2}"/>
+    </xacro:macro>
 </robot>

File: xacro/collision_objects/shelf.urdf.xacro (robot description, xacro)
@@ -1,81 +1,80 @@
 <?xml version="1.0" ?>
 <robot name="shelf" xmlns:xacro="http://www.ros.org/wiki/xacro">
-  <xacro:include filename="$(find urdf_to_scene)/xacro/planning_scene.xacro" />
-  <!-- Generic Open Shelf macro -->
-  <!-- TODO add option for an open and a closed shelf -->
-  <xacro:macro name="shelf" params="name
-                                    frame_id
-                                    xyz:='0 0 0'
-                                    rpy:='0 0 0'
-                                    dimensions:='0.6 1.5 1.25'
-                                    h_boards:=5
-                                    v_boards:=3
-                                    h_board_thickness:=0.02
-                                    v_board_thickness:=0.02
-                                    back_board:=false
-                                    dl:=_">
-  <!-- Property -->
-  <xacro:property name="root" value="${name}" />
-  <xacro:property name="hboard_gap" value="${float(dimensions.split()[2])/h_boards}" />
-  <xacro:property name="vboard_gap" value="${float(dimensions.split()[1])/(1 + v_boards)}" />
-  <xacro:property name="dim_x" value="${dimensions.split()[0]}" />
-  <xacro:property name="dim_y" value="${dimensions.split()[1]}" />
-  <xacro:property name="dim_z" value="${dimensions.split()[2]}" />
-  <xacro:property name="hboard_dim_x" value="${dim_x}" />
-  <xacro:property name="hboard_dim_y" value="${vboard_gap + v_board_thickness/2}" />
-  <xacro:property name="hboard_dim_z" value="${h_board_thickness}" />
-  <xacro:property name="hboard_dimensions" value="${hboard_dim_x} ${hboard_dim_y} ${hboard_dim_z}" />
-  <xacro:property name="vboard_dim_x" value="${dim_x}" />
-  <xacro:property name="vboard_dim_y" value="${v_board_thickness}" />
-  <xacro:property name="vboard_dim_z" value="${dim_z}" />
-  <xacro:property name="vboard_dimensions" value="${vboard_dim_x} ${vboard_dim_y} ${vboard_dim_z}" />
-  <!-- Base link -->
-  <xacro:dummy name="${root}"
-               frame_id="${frame_id}"
-               xyz="${xyz}" rpy="${rpy}" />
-  <!-- Leftmost and rightmost vertical boards -->
-  <xacro:framebox name="${root}${dl}vboard1"
-                  frame_id="${root}"
-                  dimensions="${vboard_dimensions}"
-                  xyz="0 ${-(dim_y/2 - v_board_thickness/2)} 0"/>
-  <xacro:framebox name="${root}${dl}vboard${v_boards + 2}"
-                  frame_id="${root}"
-                  dimensions="${vboard_dimensions}"
-                  xyz="0 ${dim_y/2 - v_board_thickness/2} 0"/>
-  <!-- Vertical inside boards -->
-  <xacro:macro name="loopvboard" params="current:=0 until:=^">
-    <xacro:if value="${until > current}">
-      <xacro:framebox name="${root}${dl}vboard${current+2}"
-                      frame_id="${root}${dl}vboard1/bottom"
-                      dimensions="${vboard_dimensions}"
-                      xyz="0 ${(current+1)*vboard_gap- v_board_thickness/2} 0"/>
-      <xacro:loopvboard current="${current+1}"/>
+    <xacro:include filename="$(find urdf_to_scene)/xacro/planning_scene.xacro" />
+    <!-- Generic shelf macro -->
+    <xacro:macro name="shelf" params="name
+                                      frame_id
+                                      xyz:='0 0 0'
+                                      rpy:='0 0 0'
+                                      dimensions:='0.6 1.5 1.25'
+                                      h_boards:=5
+                                      v_boards:=3
+                                      h_board_thickness:=0.02
+                                      v_board_thickness:=0.02
+                                      back_board:=false
+                                      dl:='_'">
+    <!-- Properties -->
+    <xacro:property name="root" value="${name}" />
+    <xacro:property name="hboard_gap" value="${float(dimensions.split()[2])/h_boards}" />
+    <xacro:property name="vboard_gap" value="${float(dimensions.split()[1])/(1 + v_boards)}" />
+    <xacro:property name="dim_x" value="${dimensions.split()[0]}" />
+    <xacro:property name="dim_y" value="${dimensions.split()[1]}" />
+    <xacro:property name="dim_z" value="${dimensions.split()[2]}" />
+    <xacro:property name="hboard_dim_x" value="${dim_x}" />
+    <xacro:property name="hboard_dim_y" value="${vboard_gap + v_board_thickness/2}" />
+    <xacro:property name="hboard_dim_z" value="${h_board_thickness}" />
+    <xacro:property name="hboard_dimensions" value="${hboard_dim_x} ${hboard_dim_y} ${hboard_dim_z}" />
+    <xacro:property name="vboard_dim_x" value="${dim_x}" />
+    <xacro:property name="vboard_dim_y" value="${v_board_thickness}" />
+    <xacro:property name="vboard_dim_z" value="${dim_z}" />
+    <xacro:property name="vboard_dimensions" value="${vboard_dim_x} ${vboard_dim_y} ${vboard_dim_z}" />
+    <!-- Base link -->
+    <xacro:frame name="${root}"
+                 frame_id="${frame_id}"
+                 xyz="${xyz}" rpy="${rpy}" />
+    <!-- Leftmost and rightmost vertical boards -->
+    <xacro:collision_box name="${root}${dl}vboard1"
+                         frame_id="${root}"
+                         dimensions="${vboard_dimensions}"
+                         xyz="0 ${-(dim_y/2 - v_board_thickness/2)} ${dim_z/2}"/>
+    <xacro:collision_box name="${root}${dl}vboard${v_boards + 2}"
+                         frame_id="${root}"
+                         dimensions="${vboard_dimensions}"
+                         xyz="0 ${dim_y/2 - v_board_thickness/2} ${dim_z/2}"/>
+    <!-- Vertical inside boards -->
+    <xacro:macro name="loopvboard" params="current:=0 until:=^">
+        <xacro:if value="${until > current}">
+            <xacro:collision_box name="${root}${dl}vboard${current+2}"
+                                 frame_id="${root}${dl}vboard1"
+                                 dimensions="${vboard_dimensions}"
+                                 xyz="0 ${(current+1)*vboard_gap- v_board_thickness/2} 0"/>
+            <xacro:loopvboard current="${current+1}"/>
+        </xacro:if>
+    </xacro:macro>
+    <xacro:loopvboard until="${v_boards}"/>
+    <!-- Horizontal boards -->
+    <xacro:macro name="loophboard" params="current:=0 index:=^ until:=^">
+        <xacro:if value="${until > current}">
+            <xacro:collision_box name="${root}${dl}board${index*h_boards+current+1}"
+                                 frame_id="${root}${dl}vboard${index+1}"
+                                 dimensions="${hboard_dimensions}"
+                                 xyz="0 ${(vboard_gap - v_board_thickness/2)/2} ${(current + 1)*hboard_gap - h_board_thickness/2 - dim_z/2}"/>
+            <xacro:loophboard current="${current+1}"/>
+        </xacro:if>
+    </xacro:macro>
+    <xacro:macro name="loophrowboard" params="current:=0 until:=^">
+        <xacro:if value="${until > current}">
+            <xacro:loophboard index="${current}" until="${h_boards}"/>
+            <xacro:loophrowboard current="${current+1}"/>
+        </xacro:if>
+    </xacro:macro>
+    <xacro:loophrowboard until="${v_boards + 1}"/>
+    <!-- Back board -->
+    <xacro:if value="${back_board}">
+        <xacro:collision_box name="${root}${dl}backboard"
+                             frame_id="${root}"
+                             dimensions="${v_board_thickness} ${dim_y} ${dim_z}"
+                             xyz="${-dim_x/2} 0 0"/>
     </xacro:if>
-  </xacro:macro>
-  <xacro:loopvboard until="${v_boards}"/>
-  <!-- Horizontal boards -->
-  <xacro:macro name="loophboard" params="current:=0 index:=^ until:=^">
-    <xacro:if value="${until > current}">
-      <xacro:framebox name="${root}${dl}board${index*h_boards+current+1}"
-                 frame_id="${root}${dl}vboard${index+1}/bottom"
-                 dimensions="${hboard_dimensions}"
-                 xyz="0 ${(vboard_gap - v_board_thickness/2)/2} ${(current + 1)*hboard_gap - h_board_thickness}"/>
-      <xacro:loophboard current="${current+1}"/>
-    </xacro:if>
-  </xacro:macro>
-  <xacro:macro name="loophrowboard" params="current:=0 until:=^">
-    <xacro:if value="${until > current}">
-      <xacro:loophboard index="${current}" until="${h_boards}"/>
-      <xacro:loophrowboard current="${current+1}"/>
-    </xacro:if>
-  </xacro:macro>
-  <xacro:loophrowboard until="${v_boards + 1}"/>
-  <!-- Back board -->
-  <xacro:if value="${back_board}">
-    <xacro:framebox name="${root}${dl}backboard"
-                    frame_id="${root}"
-                    dimensions="${v_board_thickness} ${dim_y} ${dim_z}"
-                    xyz="${-dim_x/2} 0 0"/>
-  </xacro:if>
-  </xacro:macro>
+    </xacro:macro>
 </robot>
