Commit message: Reformat Xacro macro planning scene API
Add descriptive macro names and comments. Update object collection.

File: xacro/planning_scene.xacro (robot description, xacro)
@@ -1,111 +1,126 @@
 <?xml version="1.0" ?>
-<robot xmlns:xacro="http://www.ros.org/wiki/xacro" name="panda">
-  <!-- Utility macros for creating collision objects as URDF -->
-  <!-- Store tf information as a joint for the collision object -->
-  <xacro:macro name="tf" params="name parent *origin">
-    <joint name="${name}" type="fixed">
-      <xacro:insert_block name="origin" />
-      <parent link="${parent}" />
-      <child link="${name}" />
-      <axis xyz="0 0 1" />
-    </joint>
-  </xacro:macro>
-  <!-- Add dummy link with no collision -->
-  <xacro:macro name="dummy" params="name frame_id xyz:='0 0 0' rpy:='0 0 0'">
-    <link name="${name}"/>
-    <xacro:tf name="${name}" parent="${frame_id}">
-      <origin xyz="${xyz}" rpy="${rpy}"/>
-    </xacro:tf>
-  </xacro:macro>
-  <!-- Add subframes for mesh -->
-  <xacro:macro name="loopmeshsubframes" params="current:=0 until:=^ node:=^ sorted_keys:=^ name:=^">
-    <xacro:if value="${until > current}">
-      <xacro:property name="xyz" value="0 0 0" />
-      <xacro:property name="rpy" value="0 0 0" />
-      <xacro:if value="${'xyz' in node[sorted_keys[current]]}">
-        <xacro:property name="xyz" value="${node[sorted_keys[current]]['xyz'][0]} ${node[sorted_keys[current]]['xyz'][1]} ${node[sorted_keys[current]]['xyz'][2]}" />
-      </xacro:if>>
-      <xacro:if value="${'rpy' in node[sorted_keys[current]]}">
-        <xacro:property name="rpy" value="${node[sorted_keys[current]]['rpy'][0]} ${node[sorted_keys[current]]['rpy'][1]} ${node[sorted_keys[current]]['rpy'][2]}" />
-      </xacro:if>
-      <xacro:subframe name="${name}"
-                      subframe="${sorted_keys[current]}"
-                      frame_id="${name}"
-                      xyz="${xyz}" rpy="${rpy}" />
-      <xacro:loopmeshsubframes current="${current+1}"/>
-    </xacro:if>
-  </xacro:macro>
-  <!-- Add mesh -->
-  <xacro:macro name="framemesh" params="name frame_id metadata xyz:='0 0 0' rpy:='0 0 0' scale:='1.0 1.0 1.0'">
-    <link name="${name}">
-      <collision>
-        <geometry>
-          <mesh filename="${metadata['resource']}" scale="${scale}" />
-        </geometry>
-      </collision>
-    </link>
-    <xacro:tf name="${name}" parent="${frame_id}">
-      <origin xyz="${xyz}" rpy="${rpy}"/>
-    </xacro:tf>
-    <xacro:if value="${'subframes' in metadata}">
-      <xacro:loopmeshsubframes until="${len(metadata['subframes'])}" node="${metadata['subframes']}" sorted_keys="${sorted(metadata['subframes'])}"/>
-    </xacro:if>
-  </xacro:macro>
-  <!-- Add primitive box -->
-  <xacro:macro name="framebox" params="name frame_id dimensions xyz:='0 0 0' rpy:='0 0 0'">
-    <!-- Parent joint -->
-    <xacro:tf name="${name}" parent="${frame_id}">
-      <!-- Add fixed origin and include z dimension -->
-      <origin xyz="${xyz.split()[0]} ${xyz.split()[1]} ${float(xyz.split()[2]) + float(dimensions.split()[2])}"/>
-    </xacro:tf>
-    <!-- Child link -->
-    <link name="${name}">
-      <collision>
-        <!-- Replace collision visualization because box origin is in the middle -->
-        <origin xyz="0 0 ${-float(dimensions.split()[2])/2}" rpy="${rpy}"/>
-        <geometry>
-          <box size="${dimensions}" />
-        </geometry>
-      </collision>
-    </link>
-    <xacro:subframe name="${name}"
-                    subframe="bottom"
-                    frame_id="${name}"
-                    xyz="0 0 ${-float(dimensions.split()[2])}" />
-    <xacro:subframe name="${name}"
-                    subframe="top"
-                    frame_id="${name}"
-                    xyz="0 0 ${float(dimensions.split()[2])}" />
-    <xacro:subframe name="${name}"
-                    subframe="back"
-                    frame_id="${name}"
-                    xyz="${-float(dimensions.split()[0])/2} 0 0" />
-    <xacro:subframe name="${name}"
-                    subframe="front"
-                    frame_id="${name}"
-                    xyz="${float(dimensions.split()[0])/2} 0 0" />
-    <xacro:subframe name="${name}"
-                    subframe="left"
-                    frame_id="${name}"
-                    xyz="0 ${-float(dimensions.split()[1])/2} 0" />
-    <xacro:subframe name="${name}"
-                    subframe="right"
-                    frame_id="${name}"
-                    xyz="0 ${float(dimensions.split()[1])/2} 0" />
-  </xacro:macro>
-  <!-- Add subframe -->
-  <!-- Optional: frame_id defaults to name parameter if empty -->
-  <xacro:macro name="subframe" params="name subframe frame_id:='' dl:=/ xyz:='0 0 0' rpy:='0 0 0'">
-    <link name="${name}${dl}${subframe}"/>
-    <xacro:if value="${len(frame_id) > 0}">
-      <xacro:tf name="${name}${dl}${subframe}" parent="${frame_id}">
-        <origin xyz="${xyz}" rpy="${rpy}"/>
-      </xacro:tf>
-    </xacro:if>
-    <xacro:unless value="${len(frame_id) > 0}">
-      <xacro:tf name="${name}${dl}${subframe}" parent="${name}">
-        <origin xyz="${xyz}" rpy="${rpy}"/>
-      </xacro:tf>
-    </xacro:unless>
-  </xacro:macro>
+<!-- Collection of macros for creating a MoveIt PlanningScene from a URDF representation -->
+<robot xmlns:xacro="http://www.ros.org/wiki/xacro" name="planning_scene">
+    <!-- TF stored in the urdf joint, used internally -->
+    <xacro:macro name="_tf" params="name parent *origin">
+        <joint name="${name}" type="fixed">
+            <xacro:insert_block name="origin" />
+            <parent link="${parent}" />
+            <child link="${name}" />
+        </joint>
+    </xacro:macro>
+    <!-- TF for building collision objects as urdf -->
+    <!-- WARNING Looses meaning upon conversion -->
+    <xacro:macro name="frame" params="name frame_id xyz:='0 0 0' rpy:='0 0 0'">
+        <!-- Empty link necessary to differentiate from other collision objects -->
+        <link name="${name}"/>
+        <xacro:_tf name="${name}" parent="${frame_id}">
+            <origin xyz="${xyz}" rpy="${rpy}"/>
+        </xacro:_tf>
+    </xacro:macro>
+    <!-- Subframe acts like the 'frame' macro, except that the tf is stored in the subframe upon conversion -->
+    <!-- WARNING Converts to a subframe only with MoveIt >= 1.0.1 -->
+    <xacro:macro name="subframe" params="name subframe_name frame_id xyz:='0 0 0' rpy:='0 0 0' dl:=/">
+        <!-- Empty link necessary to differentiate from other collision objects -->
+        <!-- Delimiter in name to differentiate from the 'frame' macro -->
+        <link name="${name}${dl}${subframe_name}"/>
+        <xacro:_tf name="${name}${dl}${subframe_name}" parent="${frame_id}">
+            <origin xyz="${xyz}" rpy="${rpy}"/>
+        </xacro:_tf>
+    </xacro:macro>
+    <!-- Box collision object -->
+    <xacro:macro name="collision_box" params="name frame_id dimensions xyz:='0 0 0' rpy:='0 0 0' scale:='1.0 1.0 1.0' default_subframes:=True">
+        <!-- Collision object stored as a urdf link -->
+        <link name="${name}">
+            <!-- Box shape -->
+            <collision>
+                <geometry>
+                    <box size="${dimensions}" />
+                </geometry>
+            </collision>
+        </link>
+        <!-- Collision object frame -->
+        <xacro:_tf name="${name}" parent="${frame_id}">
+            <origin xyz="${xyz}" rpy="${rpy}"/>
+        </xacro:_tf>
+        <!-- Add default subframes (front, back, left, right, top, down) -->
+        <xacro:_bb_subframes name="${name}"
+                            bbx="${float(dimensions.split()[0])/2}"
+                            bby="${float(dimensions.split()[1])/2}"
+                            bbz="${float(dimensions.split()[2])/2}"/>
+    </xacro:macro>
+    <!-- Cylinder collision object -->
+    <xacro:macro name="collision_cylinder" params="name frame_id radius length xyz:='0 0 0' rpy:='0 0 0' scale:='1.0 1.0 1.0'">
+        <link name="${name}">
+            <collision>
+                <geometry>
+                    <cylinder radius="${radius}" length="${length}"/>
+                </geometry>
+            </collision>
+        </link>
+        <xacro:_tf name="${name}" parent="${frame_id}">
+            <origin xyz="${xyz}" rpy="${rpy}"/>
+        </xacro:_tf>
+        <xacro:_bb_subframes name="${name}"
+                            bbx="${float(dimensions.split()[0])/2}"
+                            bby="${float(dimensions.split()[1])/2}"
+                            bbz="${float(dimensions.split()[2])/2}"/>
+    </xacro:macro>
+    <!-- Sphere collision object -->
+    <xacro:macro name="collision_sphere" params="name frame_id radius xyz:='0 0 0' rpy:='0 0 0' scale:='1.0 1.0 1.0'">
+        <link name="${name}">
+            <collision>
+                <geometry>
+                    <sphere radius="${radius}" />
+                </geometry>
+            </collision>
+        </link>
+        <xacro:_tf name="${name}" parent="${frame_id}">
+            <origin xyz="${xyz}" rpy="${rpy}"/>
+        </xacro:_tf>
+        <xacro:_bb_subframes name="${name}"
+                            bbx="${float(dimensions.split()[0])/2}"
+                            bby="${float(dimensions.split()[1])/2}"
+                            bbz="${float(dimensions.split()[2])/2}"/>
+    </xacro:macro>
+    <!-- Mesh collision object -->
+    <xacro:macro name="collision_mesh" params="name frame_id resource xyz:='0 0 0' rpy:='0 0 0' scale:='1.0 1.0 1.0'">
+        <link name="${name}">
+            <collision>
+                <geometry>
+                    <mesh filename="${resource}" scale="${scale}" />
+                </geometry>
+            </collision>
+        </link>
+        <xacro:_tf name="${name}" parent="${frame_id}">
+            <origin xyz="${xyz}" rpy="${rpy}"/>
+        </xacro:_tf>
+    </xacro:macro>
+    <!-- Default bounding box information as subframes, used internally -->
+    <xacro:macro name="_bb_subframes" params="name bbx bby bbz">
+        <xacro:subframe name="${name}"
+                        subframe_name="bottom"
+                        frame_id="${name}"
+                        xyz="0 0 ${-float(bbz)}" />
+        <xacro:subframe name="${name}"
+                        subframe_name="top"
+                        frame_id="${name}"
+                        xyz="0 0 ${float(bbz)}" />
+        <xacro:subframe name="${name}"
+                        subframe_name="back"
+                        frame_id="${name}"
+                        xyz="${-float(bbx)} 0 0" />
+        <xacro:subframe name="${name}"
+                        subframe_name="front"
+                        frame_id="${name}"
+                        xyz="${float(bbx)} 0 0" />
+        <xacro:subframe name="${name}"
+                        subframe_name="left"
+                        frame_id="${name}"
+                        xyz="0 ${-float(bby)} 0" />
+        <xacro:subframe name="${name}"
+                        subframe_name="right"
+                        frame_id="${name}"
+                        xyz="0 ${float(bby)} 0" />
+    </xacro:macro>
 </robot>
