Commit message: Compute collision_mesh subframes from metadata dictionary
Add new optional 'metadata' attribute to automatically add subframes of a 'collision_mesh' macro.

File: xacro/planning_scene.xacro (robot description, xacro)
@@ -85,5 +85,5 @@
     </xacro:macro>
     <!-- Mesh collision object -->
-    <xacro:macro name="collision_mesh" params="name frame_id resource xyz:='0 0 0' rpy:='0 0 0' scale:='1.0 1.0 1.0'">
+    <xacro:macro name="collision_mesh" params="name frame_id resource metadata:='{}' xyz:='0 0 0' rpy:='0 0 0' scale:='1.0 1.0 1.0'">
         <link name="${name}">
             <collision>
@@ -96,4 +96,15 @@
             <origin xyz="${xyz}" rpy="${rpy}"/>
         </xacro:_tf>
+        <!-- Add bounding box subframes from metadata -->
+        <xacro:if value="${'bb' in metadata}">
+            <xacro:_bb_subframes name="${name}"
+                                bbx="${float(metadata['bb'][0])/2}"
+                                bby="${float(metadata['bb'][1])/2}"
+                                bbz="${float(metadata['bb'][2])/2}"/>
+        </xacro:if>
+        <!-- Add subframes from metadata -->
+        <xacro:if value="${'subframes' in metadata}">
+            <xacro:loop name="${name}" keys="${list(metadata['subframes'].keys())}" values="${list(metadata['subframes'].values())}"/>
+        </xacro:if>
     </xacro:macro>
     <!-- Default bounding box information as subframes, used internally -->
@@ -124,3 +135,27 @@
                         xyz="0 ${float(bby)} 0" />
     </xacro:macro>
+    <!-- Loop for adding custom subframes metadata -->
+    <xacro:macro name="loop" params="name:=^ keys:=^ values:=^">
+        <xacro:if value="${keys}">
+            <!-- pop first item from list -->
+            <xacro:property name="key" value="${keys.pop(0)}"/>
+            <xacro:property name="val" value="${values.pop(0)}"/>
+            <!-- extract pose -->
+            <xacro:property name="xyz" value="0 0 0" />
+            <xacro:property name="rpy" value="0 0 0" />
+            <xacro:if value="${'xyz' in val}">
+                 <xacro:property name="xyz" value="${val['xyz'][0]} ${val['xyz'][1]} ${val['xyz'][2]}"/>
+            </xacro:if>
+            <xacro:if value="${'rpy' in val}">
+                 <xacro:property name="rpy" value="${val['rpy'][0]} ${val['rpy'][1]} ${val['rpy'][2]}"/>
+            </xacro:if>
+            <xacro:subframe name="${name}"
+                            subframe_name="${key}"
+                            frame_id="${name}"
+                            xyz="${xyz}"
+                            rpy="${rpy}"/>
+            <!-- recursively call myself -->
+            <xacro:loop/>
+        </xacro:if>
+    </xacro:macro>
 </robot>

Commit message: Remove scale option for primitive shapes

File: xacro/planning_scene.xacro (robot description, xacro)
@@ -30,5 +30,5 @@
     </xacro:macro>
     <!-- Box collision object -->
-    <xacro:macro name="collision_box" params="name frame_id dimensions xyz:='0 0 0' rpy:='0 0 0' scale:='1.0 1.0 1.0' default_subframes:=True">
+    <xacro:macro name="collision_box" params="name frame_id dimensions xyz:='0 0 0' rpy:='0 0 0' default_subframes:=True">
         <!-- Collision object stored as a urdf link -->
         <link name="${name}">
@@ -51,5 +51,5 @@
     </xacro:macro>
     <!-- Cylinder collision object -->
-    <xacro:macro name="collision_cylinder" params="name frame_id radius length xyz:='0 0 0' rpy:='0 0 0' scale:='1.0 1.0 1.0'">
+    <xacro:macro name="collision_cylinder" params="name frame_id radius length xyz:='0 0 0' rpy:='0 0 0'">
         <link name="${name}">
             <collision>
@@ -68,5 +68,5 @@
     </xacro:macro>
     <!-- Sphere collision object -->
-    <xacro:macro name="collision_sphere" params="name frame_id radius xyz:='0 0 0' rpy:='0 0 0' scale:='1.0 1.0 1.0'">
+    <xacro:macro name="collision_sphere" params="name frame_id radius xyz:='0 0 0' rpy:='0 0 0'">
         <link name="${name}">
             <collision>

Commit message: Add option to convert a `collision_box` to a mesh box

File: xacro/planning_scene.xacro (robot description, xacro)
@@ -30,19 +30,33 @@
     </xacro:macro>
     <!-- Box collision object -->
-    <xacro:macro name="collision_box" params="name frame_id dimensions xyz:='0 0 0' rpy:='0 0 0' default_subframes:=True">
-        <!-- Collision object stored as a urdf link -->
-        <link name="${name}">
-            <!-- Box shape -->
-            <collision>
-                <geometry>
-                    <box size="${dimensions}" />
-                </geometry>
-            </collision>
-        </link>
-        <!-- Collision object frame -->
-        <xacro:_tf name="${name}" parent="${frame_id}">
-            <origin xyz="${xyz}" rpy="${rpy}"/>
-        </xacro:_tf>
+    <xacro:macro name="collision_box" params="name frame_id dimensions xyz:='0 0 0' rpy:='0 0 0' mesh_resource:='' default_subframes:=True">
+        <!-- convert to a `shape_msgs/SolidPrimitive` -->
+        <xacro:if value="${len(mesh_resource) == 0}">
+            <!-- Collision object stored as a urdf link -->
+            <link name="${name}">
+                <!-- Box shape -->
+                <collision>
+                    <geometry>
+                        <box size="${dimensions}" />
+                    </geometry>
+                </collision>
+            </link>
+            <!-- Collision object frame -->
+            <xacro:_tf name="${name}" parent="${frame_id}">
+                <origin xyz="${xyz}" rpy="${rpy}"/>
+            </xacro:_tf>
+        </xacro:if>
+        <!-- convert to a `shape_msgs/Mesh.msg` -->
+        <xacro:unless value="${len(mesh_resource) == 0}">
+            <!-- apply dimensions on scale, must use a unit mesh -->
+            <xacro:collision_mesh name="${name}"
+                                  frame_id="${frame_id}"
+                                  xyz="${xyz}"
+                                  rpy="${rpy}"
+                                  resource="${mesh_resource}"
+                                  scale="${dimensions}"/>
+        </xacro:unless>
         <!-- Add default subframes (front, back, left, right, top, down) -->
+        <!-- Warning :if usin a mesh resource, the origin MUST be located in the center -->
         <xacro:_bb_subframes name="${name}"
                              bbx="${float(dimensions.split()[0])/2}"
